File: DaESK_TH1.kicad_pcb (KiCad board)
At the start: 2 copper layers, 96.8 x 94.7 mm, 36 parts, among them J1 Mousebite 8, J10 Mousebite 5, J2 Mousebite 10, J3 Mousebite 4, J4 Mousebite 10, J5 Mousebite 5, J6 Conn_01x11, J7 Mousebite 4, J8 Mousebite 4, J9 Conn_01x06

Commit message: pcb udated
Parts:
- J10: renamed from J3; footprint Keyboard-Library:mousebite4 -> Keyboard Library:mousebite4
- J5: renamed from J1; footprint Keyboard-Library:mousebite8 -> Keyboard Library:mousebite8
- J6: renamed from J5; footprint Keyboard-Library:mousebite5 -> Keyboard Library:mousebite5
- J7: renamed from J10; footprint Keyboard-Library:mousebite5 -> Keyboard Library:mousebite5
- J8: renamed from J7; footprint Keyboard-Library:mousebite4 -> Keyboard Library:mousebite4
- J9: renamed from J8; footprint Keyboard-Library:mousebite4 -> Keyboard Library:mousebite4
- RGB_TH1R1, RGB_TH1R2, RGB_TH1R3, RGB_TH1R4, RGB_TH2R1, RGB_TH2R2, RGB_TH2R3, RGB_TH2R4: footprint Keyboard 2:LEDSC160X160X070-4N_reversible -> Keyboard Library:LEDSC160X160X070-4N_reversible
- ST1: footprint keyswitches:Stabilizer_MX_2u -> Keyboard Library:Stabilizer_MX_2u
- TH1_R1, TH1_R2, TH1_R3, TH1_R4, TH2_R2, TH2_R3, TH2_R4: footprint Keyboard 2:Kailh_socket_MX_reversible_v2 -> Keyboard Library:Kailh_socket_MX_reversible_v2
- TH2_R1: footprint Keyboard 2:Kailh_socket_MX_reversible_v2_2u -> Keyboard Library:Kailh_socket_MX_reversible_v2_2u
- renumbered D9 to D1, D10 to D2, J6 to J1, J9 to J2, J2 to J3
