File: thumb_1.sch (KiCad schematic (older format))
At the start: 28 parts, among them J1 Mousebite 10, J2 Mousebite 10, J3 Mousebite 8, J4 Mousebite 5, J5 Mousebite 5, J6 Conn_01x11, J6 Mousebite 4, J7 Mousebite 4, J8 Mousebite 4, J9 Conn_01x06

Commit message: pcb udated
Parts:
- J10: renamed from J8; footprint Keyboard-Library:mousebite4 -> Keyboard Library:mousebite4
- J5: renamed from J3; footprint Keyboard-Library:mousebite8 -> Keyboard Library:mousebite8
- J6: renamed from J4; footprint Keyboard-Library:mousebite5 -> Keyboard Library:mousebite5
- J7: renamed from J5; footprint Keyboard-Library:mousebite5 -> Keyboard Library:mousebite5
- J8: renamed from J6; footprint Keyboard-Library:mousebite4 -> Keyboard Library:mousebite4
- J9: renamed from J7; footprint Keyboard-Library:mousebite4 -> Keyboard Library:mousebite4
- renumbered J1 to J3, J2 to J4
