File: DaESK-4R.sch (KiCad schematic (older format))
At the start: 7 parts

Commit message: 4R updated placement of MCU
Parts:
- H1, H2, H3, H4, H5, H6, H7: Fält4 (none) -> 0; Manufacturer_Part_Number (none) -> Hole
Changed lines of the file:
@@
 Sheet 1 4
 Title "Da.E.S.K.4R - Dual axis Ergo Split Keyboard 4 Row"
-Date "2020-09-29"
-Rev "0.91"
+Date "2020-10-13"
+Rev "0.95"
 Comp "Markus Knutsson <markus.knutsson@tweety.se>"
 Comment1 "https://github.com/TweetyDaBird"
@@
 F 2 "MountingHole:MountingHole_3.7mm" H 2300 3750 50  0001 C CNN
 F 3 "~" H 2300 3750 50  0001 C CNN
+F 4 "0" H 2300 3750 50  0001 C CNN "Fält4"
+F 5 "Hole" H 2300 3750 50  0001 C CNN "Manufacturer_Part_Number"
 	1    2300 3750
 	1    0    0    -1
@@
 F 2 "MountingHole:MountingHole_3.7mm" H 2300 3950 50  0001 C CNN
 F 3 "~" H 2300 3950 50  0001 C CNN
+F 4 "0" H 2300 3950 50  0001 C CNN "Fält4"
+F 5 "Hole" H 2300 3950 50  0001 C CNN "Manufacturer_Part_Number"
 	1    2300 3950
 	1    0    0    -1
@@
 F 2 "MountingHole:MountingHole_3.7mm" H 3150 4150 50  0001 C CNN
 F 3 "~" H 3150 4150 50  0001 C CNN
+F 4 "0" H 3150 4150 50  0001 C CNN "Fält4"
+F 5 "Hole" H 3150 4150 50  0001 C CNN "Manufacturer_Part_Number"
 	1    3150 4150
 	1    0    0    -1
@@
 F 2 "MountingHole:MountingHole_3.7mm" H 3150 3950 50  0001 C CNN
 F 3 "~" H 3150 3950 50  0001 C CNN
+F 4 "0" H 3150 3950 50  0001 C CNN "Fält4"
+F 5 "Hole" H 3150 3950 50  0001 C CNN "Manufacturer_Part_Number"
 	1    3150 3950
 	1    0    0    -1
@@
 F 2 "MountingHole:MountingHole_3.7mm" H 3150 3750 50  0001 C CNN
 F 3 "~" H 3150 3750 50  0001 C CNN
+F 4 "0" H 3150 3750 50  0001 C CNN "Fält4"
+F 5 "Hole" H 3150 3750 50  0001 C CNN "Manufacturer_Part_Number"
 	1    3150 3750
 	1    0    0    -1
@@
 F 2 "MountingHole:MountingHole_2.2mm_M2" H 2800 4350 50  0001 C CNN
 F 3 "~" H 2800 4350 50  0001 C CNN
+F 4 "0" H 2800 4350 50  0001 C CNN "Fält4"
+F 5 "Hole" H 2800 4350 50  0001 C CNN "Manufacturer_Part_Number"
 	1    2800 4350
 	1    0    0    -1
@@
 F 2 "MountingHole:MountingHole_3.7mm" H 2300 4150 50  0001 C CNN
 F 3 "~" H 2300 4150 50  0001 C CNN
+F 4 "0" H 2300 4150 50  0001 C CNN "Fält4"
+F 5 "Hole" H 2300 4150 50  0001 C CNN "Manufacturer_Part_Number"
 	1    2300 4150
 	1    0    0    -1
