File: RGB_array_4R.sch (KiCad schematic (older format))
At the start: 24 parts

Commit message: 4R updated placement of MCU
Parts:
- RGB_C2R1: value 5-ABC -> RGB; footprint Keyboard 2:LEDSC160X160X070-4N_reversible -> Keyboard Library:LEDSC160X160X070-4N_reversible; Fält4 (none) -> 1; Mouser Part Number (none) -> 604-APTF1616SEJ3ZGGV
- RGB_C2R2: value 6-ABC -> RGB; footprint Keyboard 2:LEDSC160X160X070-4N_reversible -> Keyboard Library:LEDSC160X160X070-4N_reversible; Fält4 (none) -> 1; Mouser Part Number (none) -> 604-APTF1616SEJ3ZGGV
- RGB_C2R3: value 7-ABC -> RGB; footprint Keyboard 2:LEDSC160X160X070-4N_reversible -> Keyboard Library:LEDSC160X160X070-4N_reversible; Fält4 (none) -> 1; Mouser Part Number (none) -> 604-APTF1616SEJ3ZGGV
- RGB_C2R4: value 8-ABC -> RGB; footprint Keyboard 2:LEDSC160X160X070-4N_reversible -> Keyboard Library:LEDSC160X160X070-4N_reversible; Fält4 (none) -> 1; Mouser Part Number (none) -> 604-APTF1616SEJ3ZGGV
- RGB_C3R1: value 9-ABC -> RGB; footprint Keyboard 2:LEDSC160X160X070-4N_reversible -> Keyboard Library:LEDSC160X160X070-4N_reversible; Fält4 (none) -> 1; Mouser Part Number (none) -> 604-APTF1616SEJ3ZGGV
- RGB_C3R2: value 10-ABC -> RGB; footprint Keyboard 2:LEDSC160X160X070-4N_reversible -> Keyboard Library:LEDSC160X160X070-4N_reversible; Fält4 (none) -> 1; Mouser Part Number (none) -> 604-APTF1616SEJ3ZGGV
- RGB_C3R3: value 11-ABC -> RGB; footprint Keyboard 2:LEDSC160X160X070-4N_reversible -> Keyboard Library:LEDSC160X160X070-4N_reversible; Fält4 (none) -> 1; Mouser Part Number (none) -> 604-APTF1616SEJ3ZGGV
- RGB_C3R4: value 12-ABC -> RGB; footprint Keyboard 2:LEDSC160X160X070-4N_reversible -> Keyboard Library:LEDSC160X160X070-4N_reversible; Fält4 (none) -> 1; Mouser Part Number (none) -> 604-APTF1616SEJ3ZGGV
- RGB_C4R1: value 1-DEF -> RGB; footprint Keyboard 2:LEDSC160X160X070-4N_reversible -> Keyboard Library:LEDSC160X160X070-4N_reversible; Fält4 (none) -> 1; Mouser Part Number (none) -> 604-APTF1616SEJ3ZGGV
- RGB_C4R2: value 2-DEF -> RGB; footprint Keyboard 2:LEDSC160X160X070-4N_reversible -> Keyboard Library:LEDSC160X160X070-4N_reversible; Fält4 (none) -> 1; Mouser Part Number (none) -> 604-APTF1616SEJ3ZGGV
- RGB_C4R3: value 3-DEF -> RGB; footprint Keyboard 2:LEDSC160X160X070-4N_reversible -> Keyboard Library:LEDSC160X160X070-4N_reversible; Fält4 (none) -> 1; Mouser Part Number (none) -> 604-APTF1616SEJ3ZGGV
- RGB_C4R4: value 4-DEF -> RGB; footprint Keyboard 2:LEDSC160X160X070-4N_reversible -> Keyboard Library:LEDSC160X160X070-4N_reversible; Fält4 (none) -> 1; Mouser Part Number (none) -> 604-APTF1616SEJ3ZGGV
- RGB_C5R1: value 5-DEF -> RGB; footprint Keyboard 2:LEDSC160X160X070-4N_reversible -> Keyboard Library:LEDSC160X160X070-4N_reversible; Fält4 (none) -> 1; Mouser Part Number (none) -> 604-APTF1616SEJ3ZGGV
- RGB_C5R2: value 6-DEF -> RGB; footprint Keyboard 2:LEDSC160X160X070-4N_reversible -> Keyboard Library:LEDSC160X160X070-4N_reversible; Fält4 (none) -> 1; Mouser Part Number (none) -> 604-APTF1616SEJ3ZGGV
- RGB_C5R3: value 7-DEF -> RGB; footprint Keyboard 2:LEDSC160X160X070-4N_reversible -> Keyboard Library:LEDSC160X160X070-4N_reversible; Fält4 (none) -> 1; Mouser Part Number (none) -> 604-APTF1616SEJ3ZGGV
- RGB_C5R4: value 8-DEF -> RGB; footprint Keyboard 2:LEDSC160X160X070-4N_reversible -> Keyboard Library:LEDSC160X160X070-4N_reversible; Fält4 (none) -> 1; Mouser Part Number (none) -> 604-APTF1616SEJ3ZGGV
- RGB_C6R1: value CB1_9 -> RGB; footprint Keyboard 2:LEDSC160X160X070-4N_reversible -> Keyboard Library:LEDSC160X160X070-4N_reversible; Fält4 (none) -> 1; Mouser Part Number (none) -> 604-APTF1616SEJ3ZGGV
- RGB_C6R2: value CB1_8 -> RGB; footprint Keyboard 2:LEDSC160X160X070-4N_reversible -> Keyboard Library:LEDSC160X160X070-4N_reversible; Fält4 (none) -> 1; Mouser Part Number (none) -> 604-APTF1616SEJ3ZGGV
- RGB_C6R3: value CB1_7 -> RGB; footprint Keyboard 2:LEDSC160X160X070-4N_reversible -> Keyboard Library:LEDSC160X160X070-4N_reversible; Fält4 (none) -> 1; Mouser Part Number (none) -> 604-APTF1616SEJ3ZGGV
- RGB_C6R4: value CB1_6 -> RGB; footprint Keyboard 2:LEDSC160X160X070-4N_reversible -> Keyboard Library:LEDSC160X160X070-4N_reversible; Fält4 (none) -> 1; Mouser Part Number (none) -> 604-APTF1616SEJ3ZGGV
- RGB_C7R1: value CB2_1 -> RGB; footprint Keyboard 2:LEDSC160X160X070-4N_reversible -> Keyboard Library:LEDSC160X160X070-4N_reversible; Fält4 (none) -> 1; Mouser Part Number (none) -> 604-APTF1616SEJ3ZGGV
- RGB_C7R2: value CB2_2 -> RGB; footprint Keyboard 2:LEDSC160X160X070-4N_reversible -> Keyboard Library:LEDSC160X160X070-4N_reversible; Fält4 (none) -> 1; Mouser Part Number (none) -> 604-APTF1616SEJ3ZGGV
- RGB_C7R3: value CB2_3 -> RGB; footprint Keyboard 2:LEDSC160X160X070-4N_reversible -> Keyboard Library:LEDSC160X160X070-4N_reversible; Fält4 (none) -> 1; Mouser Part Number (none) -> 604-APTF1616SEJ3ZGGV
- RGB_C7R4: value CB2_4 -> RGB; footprint Keyboard 2:LEDSC160X160X070-4N_reversible -> Keyboard Library:LEDSC160X160X070-4N_reversible; Fält4 (none) -> 1; Mouser Part Number (none) -> 604-APTF1616SEJ3ZGGV
