File: switch_array_4R.sch (KiCad schematic (older format))
At the start: 30 parts

Commit message: 4R updated placement of MCU
Parts:
- C2R1, C2R2, C2R3, C2R4, C3R1, C3R2, C3R3, C3R4, C4R1, C4R2, C4R3, C4R4, C5R1, C5R2, C5R3, C5R4, C6R1, C6R2, C6R3, C6R4, C7R1, C7R2, C7R3, C7R4: footprint Keyboard 2:Kailh_socket_MX_reversible_v2 -> Keyboard Library:Kailh_socket_MX_reversible_v2; Fält4 (none) -> 1; Manufacturer_Name (none) -> Kaihl; Manufacturer_Part_Number (none) -> CPG151101S11
- D1, D2, D3, D5, D6, D7: Fält4 (none) -> 1; Manufacturer_Name (none) -> Nexperia; Manufacturer_Part_Number (none) -> BAV70S,135; Mouser Part Number (none) -> 771-BAV70S135
